File: circuits_capteurs.kicad_sch (KiCad schematic)
At the start: 49 parts, among them U10 LMC6482IN, U2 INA823DT, U3 LMC6482IN, U4 INA823DT, U5 INA823DT, U7 LMC6482IN, U8 INA823DT, U9 LMC6482IN

Commit message: Re-re-buck
J'ai pris les trucs à Vincent et refait les modifs du buck converter.
Connections:
- new net: SG1. (Out), SG2. (Out)
- new net: SG5. (Out), SG6. (Out)
- new net: SG3. (Out), SG4. (Out)

Commit message: SPI_Debut
Connections:
- new net: SG1. (Out), SG2. (Out)
- new net: SG5. (Out), SG6. (Out)
- new net: SG3. (Out), SG4. (Out)

Commit message: Ajout de commentaires sur les pins inutilisés
Connections:
- new net: SG1. (Out), SG2. (Out)
- new net: SG5. (Out), SG6. (Out)
- new net: SG3. (Out), SG4. (Out)

Commit message: Renommer circuit caméra à payload
Connections:
- new net: SG1. (Out), SG2. (Out)
- new net: SG5. (Out), SG6. (Out)
- new net: SG3. (Out), SG4. (Out)

Commit message: Connexion partielle du connecteur usb
Connections:
- new net: SG1. (Out), SG2. (Out)
- new net: SG5. (Out), SG6. (Out)
- new net: SG3. (Out), SG4. (Out)

Commit message: CpateurFin
Parts:
- removed C4: 0,1uF, symbol Device:C
- removed C8: C, symbol Device:C
- removed RV10, RV9: R_Potentiometer (20k), symbol Device:R_Potentiometer
- removed RV4: R_Potentiometer (10k), symbol Device:R_Potentiometer
- removed U2, U4, U5, U8: INA823DT, D0008A_SOIC_TEX, symbol GAUL-Symboles:INA823DT
- added C16, C17: 10nF, symbol Device:C
- added R27, R28, R31: 800, symbol Device:R
- added R29: 1k, symbol Device:R
- added R30: 400, symbol Device:R
- added R32: 100k, symbol Device:R
- added RV11: R_Potentiometer (10k), symbol Device:R_Potentiometer
- added U13, U2: INA2331AIPWR, PW14, symbol GAUL-Symboles:INA2331AIPWR
- C1, C5: value 0,1uF -> 10nF
- C2: value 0.1uF -> 10nF
- C6, C7: value C -> 10nF
- R1: value 9k -> 8k
- R11: value 16k -> 10k
- R13: value 2k -> 100k
- R15, R16, R17: value R -> 1k
- R20: value 1k -> 10k
- R4, R5: value 20k -> 22k
- R6, R8: value 1k -> 100k
- RV8: value R_Potentiometer (20k) -> R_Potentiometer (10k)
Connections:
- net ADC1: now also R13.2
- net ADC2: now also R32.2
- net GND: now also R15.2, R16.2, R17.2, RV5.3, C16.2, C17.2, R29.2, RV11.3, U13.10 (REFB), U13.12 (REFA), U13.4 (V-), U2.10 (REFB), U2.12 (REFA), U2.4 (V-)
- net IN+: now also U13.3 (VIN+A)
- net IN-: now also U13.2 (VIN-A), U13.5 (VIN+B), U2.2 (VIN-A)
- net IN1+: now also U13.6 (VIN-B)
- net IN2+: now also U2.3 (VIN+A)
- net Suiveur: now also C16.1, R27.2; no longer C6.1, R15.2
- net Suiveur1: now also C17.1, R28.2; no longer C7.1, R16.2
- net Suiveur2: now also C7.1, R31.2; no longer R17.2
- net out+: now also U2.5 (VIN+B)
- net out-: now also U2.6 (VIN-B)
- net at R13.1: now also C2.1, R8.2, U3.6 (NEGB)
- net Suiveur3: now reaches U9.3 (POSA)
- net Suiveur3: now also C6.1, R30.2; no longer R13.2
- net at R16.1: now also U13.1 (RGA)
- net at RV6.1: now also RV6.2, R28.1, U13.9 (VOUTB)
- net at RV6.3: now also R15.1, U13.7 (RGB); no longer RV6.2
- net at C1.1, R6.2, U3.2 (NEGA): now also R32.1
- net at RV7.1: now also RV7.2, R30.1, U2.9 (VOUTB)
- net at R17.1: now also U2.1 (RGA)
- net at RV7.3: now also R29.1, U2.7 (RGB); no longer RV7.2
- net at RV5.1: now also RV5.2, R27.1, U13.13 (VOUTA)
- net +5V renamed +3.3V
- net +3.3V: now also U13.11 (V+), U2.11 (V+)
- new net: R31.1, RV11.1, RV11.2, U2.13 (VOUTA)
- new net: SG1. (Out), SG2. (Out)
- new net: SG5. (Out), SG6. (Out)
- new net: SG3. (Out), SG4. (Out)
- no-connect marks 0 -> 4
Other:
- note added: "F0= 1.6kHz"
- note added: "F0= 160Hz"
- note added: "F0= 20kHz"
- moved on the sheet: R1, R11, R2, R3, RV1, RV2, RV3, RV6, SG1, SG2, SG3, SG4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

Commit message: Mémoire
Parts:
- R13, R32, R6, R8: value 100k -> 200k
- R20: value 10k -> 40k
- R30: value 400 -> 800
- RV8: value R_Potentiometer (10k) -> R_Potentiometer (100k) pour reach 40k
Connections:
- new net: SG1. (Out), SG2. (Out)
- new net: SG5. (Out), SG6. (Out)
- new net: SG3. (Out), SG4. (Out)
Other:
- note added: "F0= 400 Hz"
- note added: "F0= 80Hz"
- note removed: "F0= 1.6kHz"
- note removed: "F0= 160Hz"
Changed lines of the file:
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@@
     (fill (type none))
   )
-  (text "F0= 160Hz" (at 111.76 130.81 0)
+  (text "F0= 80Hz" (at 111.76 130.81 0)
     (effects (font (size 1.27 1.27)) (justify left bottom))
   )
@@
     (effects (font (size 1.27 1.27)) (justify left bottom))
   )
-  (text "F0= 1.6kHz" (at 116.84 29.21 0)
+  (text "F0= 400 Hz" (at 116.84 29.21 0)
     (effects (font (size 1.27 1.27)) (justify left bottom))
   )
@@
       (effects (font (size 1.27 1.27)))
     )
-    (property "Value" "100k" (at 93.98 138.43 90)
+    (property "Value" "200k" (at 93.98 138.43 90)
       (effects (font (size 1.27 1.27)))
     )
@@
       (effects (font (size 1.27 1.27)))
     )
-    (property "Value" "400" (at 266.7 119.38 90)
+    (property "Value" "800" (at 266.7 119.38 90)
       (effects (font (size 1.27 1.27)))
     )
@@
       (effects (font (size 1.27 1.27)) (justify left))
     )
-    (property "Value" "10k" (at 80.01 36.83 0)
+    (property "Value" "40k" (at 80.01 36.83 0)
       (effects (font (size 1.27 1.27)) (justify left))
     )
@@
       (effects (font (size 1.27 1.27)))
     )
-    (property "Value" "100k" (at 93.98 156.21 90)
+    (property "Value" "200k" (at 93.98 156.21 90)
       (effects (font (size 1.27 1.27)))
     )
@@
       (effects (font (size 1.27 1.27)) (justify left))
     )
-    (property "Value" "100k" (at 80.01 156.21 0)
+    (property "Value" "200k" (at 80.01 156.21 0)
       (effects (font (size 1.27 1.27)) (justify left))
     )
@@
       (effects (font (size 1.27 1.27)))
     )
-    (property "Value" "R_Potentiometer (10k)" (at 101.6 43.18 90)
+    (property "Value" "R_Potentiometer (100k) pour reach 40k" (at 101.6 43.18 90)
       (effects (font (size 1.27 1.27)))
     )
@@
       (effects (font (size 1.27 1.27)) (justify left))
     )
-    (property "Value" "100k" (at 76.2 138.43 0)
-      (effects (font (size 1.27 1.27)) (justify left))
-    )
+    (property "Value" "200k" (at 76.2 138.43 0)
+      (effects (font (size 1.27 1.27)) (justify left))
+    )
