File: circuit_alimentation.kicad_sch (KiCad schematic)
At the start: 0 parts

Commit message: VDDLDO
Parts:
- added C10, C17, C9: 4,7uF, symbol Device:C
- added C11, C12, C13, C14, C15, C16: 2,2uF, symbol Device:C
- added U1: STM32-(STM32H745ZIT6), LQFP-144, symbol GAUL-Symboles:STM32-(STM32H745ZIT6)
Connections:
- new net: C15.2, C16.1
- new net: C13.2, C14.1
- new net: C11.2, C12.1
- new net +3.3V: C10.2, C17.2, C9.2, U1.105 (VDDLDO), U1.143 (VDDLDO), U1.70 (VDDLDO)
- new net GND: C10.1, C12.2, C14.2, C16.2, C17.1, C9.1, U1.104 (VSS), U1.141 (VSS), U1.69 (VSS)
- new net Vcap1(68): C11.1, U1.68 (VCAP)
- new net Vcap2(103): C13.1, U1.103 (VCAP)
- new net Vcap3(140): C15.1, U1.140 (VCAP)
Other:
- note added: "Vddldo"

Commit message: Alimentation
Parts:
- added C18, C20: 1uF, symbol Device:C
- added C19, C21, C22, C23, C24, C25, C26, C27, C28, C29, C30, C31, C32, C33, C34: 100nF, symbol Device:C
- added C35, C36, C37, C38: 4,7uF, symbol Device:C
Connections:
- net +3.3V: now also U1.106 (VDD), U1.119 (VDD), U1.129 (VDD), U1.13 (VDD), U1.144 (VDD), U1.19 (VDD), U1.32 (VDD), U1.35 (VREF+), U1.36 (VDDA), U1.42 (VDD), U1.56 (VDD), U1.7 (VDD), U1.71 (VDD), U1.79 (VDD), U1.92 (VDD), C18.2, C19.2, C20.2, C21.2, C22.2, C23.2, C24.2, C25.2, C26.2, C27.2, C28.2, C29.2, C30.2, C31.2, C32.2, C33.2, C34.2, C35.2, C36.2, C37.2, C38.2
- net GND: now also C11.2, C13.2, C15.2, U1.118 (VSS), U1.12 (VSS), U1.128 (VSS), U1.18 (VSS), U1.33 (VSS), U1.34 (VSSA), U1.41 (VSS), U1.55 (VSS), U1.6 (VSS), U1.80 (VSS), U1.89 (VSS), U1.90 (VDD50USB), U1.91 (VDD33USB), C18.1, C19.1, C20.1, C21.1, C22.1, C23.1, C24.1, C25.1, C26.1, C27.1, C28.1, C29.1, C30.1, C31.1, C32.1, C33.1, C34.1, C35.1, C36.1, C37.1, C38.1
- net Vcap1(68): now also C12.1
- net Vcap2(103): now also C14.1
- net Vcap3(140): now also C16.1
Other:
- note added: "Découplage"
- note added: "P.111: SMPS (nécessaire)"
- note added: "Voltage ADC"
- moved on the sheet: C11, C12

Commit message: Alimentation2
Parts:
- removed C15, C16: 2,2uF, symbol Device:C
- removed C17: 4,7uF, symbol Device:C
- added C39: 4,7uF 100mOhm, symbol Device:C
- added C40: 220pF, symbol Device:C
- added C41, C42: 10uF 20mOhm, symbol Device:C
- added L1: 2,2uH, symbol Device:L
Connections:
- net Vcap3(140) is gone; now on net VFBSMPS: U1.140 (VCAP)
- net +3.3V: now also U1.16 (VDDSMPS), C39.1; no longer U1.143 (VDDLDO)
- net GND: now also U1.14 (VSSSMPS), C39.2, C40.2, C41.1, C42.1
- net VLXSMPS: now reaches U1.15 (VLXSMPS)
- net VLXSMPS: now also C40.1, L1.1
- net VFBSMPS: now reaches U1.17 (VFBSMPS)
- net VFBSMPS: now also U1.143 (VDDLDO), C41.2, C42.2, L1.2
Other:
- note added: "SMPS"
- note removed: "P.111: SMPS (nécessaire)"
- moved on the sheet: C10, C11, C12, C13, C14, C18, C19, C20, C21, C22, C23, C24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
