File: Payload.kicad_sch (KiCad schematic)
At the start: 2 parts, among them J1 USB4056-03-A_REVA2, U1 STM32H745ZIT6

Commit message: MPU
Other:
- added sheet MPU (MPU.kicad_sch)
Changed lines of the file:
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@@
+    )
+  )
+  (sheet (at 16.51 97.79) (size 15.24 12.7) (fields_autoplaced)
+    (stroke (width 0.1524) (type solid))
+    (fill (color 0 0 0 0.0000))
+    (property "Sheetname" "MPU" (at 16.51 97.0784 0)
+      (effects (font (size 1.27 1.27)) (justify left bottom))
+    )
+    (property "Sheetfile" "MPU.kicad_sch" (at 16.51 111.0746 0)
+      (effects (font (size 1.27 1.27)) (justify left top))
+    )
+    (instances
+      (project "Payload"
+        (path "/5f62c44b-34ee-4720-b187-b4a520863a8a" (page "5"))
+      )
     )
   )

Commit message: capteurs Update
Other:
- moved on the sheet: J1, U1A
Changed lines of the file:
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@@
     (company "GAUL")
   )
-  (symbol (lib_id "GAUL-Symboles:STM32H745ZIT6") (at 118.11 59.69 0) (unit 1)
+  (symbol (lib_id "GAUL-Symboles:STM32H745ZIT6") (at 68.58 30.48 0) (unit 1)
     (in_bom yes) (on_board yes) (dnp no) (fields_autoplaced)
-    (property "Reference" "U1" (at 148.59 49.53 0)
+    (property "Reference" "U1" (at 99.06 20.32 0)
       (effects (font (size 1.524 1.524)))
     )
-    (property "Value" "STM32H745ZIT6" (at 148.59 52.07 0)
+    (property "Value" "STM32H745ZIT6" (at 99.06 22.86 0)
       (effects (font (size 1.524 1.524)))
     )
-    (property "Footprint" "LQFP-144" (at 118.11 59.69 0)
+    (property "Footprint" "LQFP-144" (at 68.58 30.48 0)
       (effects (font (size 1.27 1.27) italic) hide)
     )
-    (property "Datasheet" "STM32H745ZIT6" (at 118.11 59.69 0)
+    (property "Datasheet" "STM32H745ZIT6" (at 68.58 30.48 0)
       (effects (font (size 1.27 1.27) italic) hide)
     )
@@
     )
   )
-  (symbol (lib_id "GAUL-Symboles:USB4056-03-A_REVA2") (at 223.52 83.82 0) (unit 1)
+  (symbol (lib_id "GAUL-Symboles:USB4056-03-A_REVA2") (at 210.82 48.26 0) (unit 1)
     (in_bom yes) (on_board yes) (dnp no) (fields_autoplaced)
-    (property "Reference" "J1" (at 223.52 63.5 0)
+    (property "Reference" "J1" (at 210.82 27.94 0)
       (effects (font (size 1.27 1.27)))
     )
-    (property "Value" "USB4056-03-A_REVA2" (at 223.52 66.04 0)
+    (property "Value" "USB4056-03-A_REVA2" (at 210.82 30.48 0)
       (effects (font (size 1.27 1.27)))
     )
-    (property "Footprint" "USB4056-03-A_REVA2:GCT_USB4056-03-A_REVA2" (at 223.52 83.82 0)
+    (property "Footprint" "USB4056-03-A_REVA2:GCT_USB4056-03-A_REVA2" (at 210.82 48.26 0)
       (effects (font (size 1.27 1.27)) (justify bottom) hide)
     )
-    (property "Datasheet" "" (at 223.52 83.82 0)
+    (property "Datasheet" "" (at 210.82 48.26 0)
       (effects (font (size 1.27 1.27)) hide)
     )
-    (property "PARTREV" "A2" (at 223.52 83.82 0)
+    (property "PARTREV" "A2" (at 210.82 48.26 0)
       (effects (font (size 1.27 1.27)) (justify bottom) hide)
     )
-    (property "STANDARD" "Manufacturer Recommendations" (at 223.52 83.82 0)
+    (property "STANDARD" "Manufacturer Recommendations" (at 210.82 48.26 0)
       (effects (font (size 1.27 1.27)) (justify bottom) hide)
     )
-    (property "SNAPEDA_PN" "USB4056-03-A" (at 223.52 83.82 0)
+    (property "SNAPEDA_PN" "USB4056-03-A" (at 210.82 48.26 0)
       (effects (font (size 1.27 1.27)) (justify bottom) hide)
     )
-    (property "MAXIMUM_PACKAGE_HEIGHT" "3.31 mm" (at 223.52 83.82 0)
+    (property "MAXIMUM_PACKAGE_HEIGHT" "3.31 mm" (at 210.82 48.26 0)
       (effects (font (size 1.27 1.27)) (justify bottom) hide)
     )
-    (property "MANUFACTURER" "GCT" (at 223.52 83.82 0)
+    (property "MANUFACTURER" "GCT" (at 210.82 48.26 0)
       (effects (font (size 1.27 1.27)) (justify bottom) hide)
     )

Commit message: VDDLDO
Parts:
- removed J1: USB4056-03-A_REVA2, USB4056-03-A_REVA2:GCT_USB4056-03-A_REVA2, symbol GAUL-Symboles:USB4056-03-A_REVA2
- removed U1: STM32H745ZIT6, LQFP-144, symbol GAUL-Symboles:STM32H745ZIT6
- added U1: STM32-(STM32H745ZIT6), LQFP-144, symbol GAUL-Symboles:STM32-(STM32H745ZIT6)

Commit message: Alimentation2
Other:
- moved on the sheet: U1B
Changed lines of the file:
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@@
     (company "GAUL")
   )
-  (symbol (lib_id "GAUL-Symboles:STM32-(STM32H745ZIT6)") (at 124.46 53.34 0) (unit 2)
+  (symbol (lib_id "GAUL-Symboles:STM32-(STM32H745ZIT6)") (at 102.87 53.34 0) (unit 2)
     (in_bom yes) (on_board yes) (dnp no) (fields_autoplaced)
-    (property "Reference" "U1" (at 152.4 43.18 0)
+    (property "Reference" "U1" (at 130.81 43.18 0)
       (effects (font (size 1.524 1.524)))
     )
-    (property "Value" "STM32-(STM32H745ZIT6)" (at 152.4 45.72 0)
+    (property "Value" "STM32-(STM32H745ZIT6)" (at 130.81 45.72 0)
       (effects (font (size 1.524 1.524)))
     )
-    (property "Footprint" "LQFP-144" (at 124.46 53.34 0)
+    (property "Footprint" "LQFP-144" (at 102.87 53.34 0)
       (effects (font (size 1.27 1.27) italic) hide)
     )
-    (property "Datasheet" "STM32H745ZIT6" (at 124.46 53.34 0)
+    (property "Datasheet" "STM32H745ZIT6" (at 102.87 53.34 0)
       (effects (font (size 1.27 1.27) italic) hide)
     )

Commit message: SPI_Debut
Parts:
- added R10, R12, R14, R18, R19, R21, R9: 170, symbol Device:R
Connections:
- net at U1.20 (PF6): now also R9.2
- net at U1.21 (PF7): now also R10.2
- net at U1.22 (PF8): now also R12.2
- net at U1.23 (PF9): now also R14.2
- net at U1.24 (PF10): now also R18.2
- net at U1.52 (PF11): now also R19.2
- net at U1.53 (PF14): now also R21.2
Other:
- note added: "PB15: MOSI, PB14: MISO, PB13: Sck, PB12: NSS"
- note added: "PE7: IO0, PE8: IO1, PE9: IO2, PE10: IO3, PE11: NSS, PE12: SCK du quadSPI"
- moved on the sheet: U1A, U1B
Changed lines of the file:
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@@
     (company "GAUL")
   )
-  (symbol (lib_id "GAUL-Symboles:STM32-(STM32H745ZIT6)") (at 102.87 53.34 0) (unit 2)
+  (wire (pts (xy 44.45 90.17) (xy 81.28 90.17))
+    (stroke (width 0) (type default))
+  )
+  (wire (pts (xy 77.47 102.87) (xy 81.28 102.87))
+    (stroke (width 0) (type default))
+  )
+  (wire (pts (xy 64.77 97.79) (xy 81.28 97.79))
+    (stroke (width 0) (type default))
+  )
+  (wire (pts (xy 71.12 100.33) (xy 81.28 100.33))
+    (stroke (width 0) (type default))
+  )
+  (wire (pts (xy 38.1 87.63) (xy 81.28 87.63))
+    (stroke (width 0) (type default))
+  )
+  (wire (pts (xy 58.42 95.25) (xy 81.28 95.25))
+    (stroke (width 0) (type default))
+  )
+  (wire (pts (xy 50.8 92.71) (xy 81.28 92.71))
+    (stroke (width 0) (type default))
+  )
+  (text "PE7: IO0, PE8: IO1, PE9: IO2, PE10: IO3, PE11: NSS, PE12: SCK du quadSPI"
+    (at 43.18 30.48 0)
+    (effects (font (size 1.27 1.27)) (justify left bottom))
+  )
+  (text "PB15: MOSI, PB14: MISO, PB13: Sck, PB12: NSS" (at 170.18 127 0)
+    (effects (font (size 1.27 1.27)) (justify left bottom))
+  )
+  (symbol (lib_id "Device:R") (at 64.77 101.6 180) (unit 1)
+    (in_bom yes) (on_board yes) (dnp no)
+    (property "Reference" "R18" (at 59.69 100.33 0)
+      (effects (font (size 1.27 1.27)) (justify right))
+    )
+    (property "Value" "170" (at 59.69 102.87 0)
+      (effects (font (size 1.27 1.27)) (justify right))
+    )
+    (property "Footprint" "" (at 66.548 101.6 90)
+      (effects (font (size 1.27 1.27)) hide)
+    )
+    (property "Datasheet" "~" (at 64.77 101.6 0)
+      (effects (font (size 1.27 1.27)) hide)
+    )
+    (pin "2")
+    (pin "1")
+    (instances
+      (project "Payload"
+        (path "/5f62c44b-34ee-4720-b187-b4a520863a8a"
+          (reference "R18") (unit 1)
+        )
+      )
+    )
+  )
+  (symbol (lib_id "Device:R") (at 58.42 99.06 180) (unit 1)
+    (in_bom yes) (on_board yes) (dnp no)
+    (property "Reference" "R14" (at 53.34 97.79 0)
+      (effects (font (size 1.27 1.27)) (justify right))
+    )
+    (property "Value" "170" (at 53.34 100.33 0)
+      (effects (font (size 1.27 1.27)) (justify right))
+    )
+    (property "Footprint" "" (at 60.198 99.06 90)
+      (effects (font (size 1.27 1.27)) hide)
+    )
+    (property "Datasheet" "~" (at 58.42 99.06 0)
+      (effects (font (size 1.27 1.27)) hide)
+    )
+    (pin "2")
+    (pin "1")
+    (instances
+      (project "Payload"
+        (path "/5f62c44b-34ee-4720-b187-b4a520863a8a"
+          (reference "R14") (unit 1)
+        )
+      )
+    )
+  )
+  (symbol (lib_id "Device:R") (at 77.47 106.68 180) (unit 1)
+    (in_bom yes) (on_board yes) (dnp no)
+    (property "Reference" "R21" (at 72.39 105.41 0)
+      (effects (font (size 1.27 1.27)) (justify right))
+    )
+    (property "Value" "170" (at 72.39 107.95 0)
+      (effects (font (size 1.27 1.27)) (justify right))
+    )
+    (property "Footprint" "" (at 79.248 106.68 90)
+      (effects (font (size 1.27 1.27)) hide)
+    )
+    (property "Datasheet" "~" (at 77.47 106.68 0)
+      (effects (font (size 1.27 1.27)) hide)
+    )
+    (pin "2")
+    (pin "1")
+    (instances
+      (project "Payload"
+        (path "/5f62c44b-34ee-4720-b187-b4a520863a8a"
+          (reference "R21") (unit 1)
+        )
+      )
+    )
+  )
+  (symbol (lib_id "Device:R") (at 38.1 91.44 180) (unit 1)
+    (in_bom yes) (on_board yes) (dnp no)
+    (property "Reference" "R9" (at 34.29 90.17 0)
+      (effects (font (size 1.27 1.27)) (justify right))
+    )
+    (property "Value" "170" (at 33.02 92.71 0)
+      (effects (font (size 1.27 1.27)) (justify right))
+    )
+    (property "Footprint" "" (at 39.878 91.44 90)
+      (effects (font (size 1.27 1.27)) hide)
+    )
+    (property "Datasheet" "~" (at 38.1 91.44 0)
+      (effects (font (size 1.27 1.27)) hide)
+    )
+    (pin "2")
+    (pin "1")
+    (instances
+      (project "Payload"
+        (path "/5f62c44b-34ee-4720-b187-b4a520863a8a"
+          (reference "R9") (unit 1)
+        )
+      )
+    )
+  )
+  (symbol (lib_id "GAUL-Symboles:STM32-(STM32H745ZIT6)") (at 81.28 44.45 0) (unit 2)
     (in_bom yes) (on_board yes) (dnp no) (fields_autoplaced)
-    (property "Reference" "U1" (at 130.81 43.18 0)
+    (property "Reference" "U1" (at 109.22 34.29 0)
       (effects (font (size 1.524 1.524)))
     )
-    (property "Value" "STM32-(STM32H745ZIT6)" (at 130.81 45.72 0)
+    (property "Value" "STM32-(STM32H745ZIT6)" (at 109.22 36.83 0)
       (effects (font (size 1.524 1.524)))
     )
-    (property "Footprint" "LQFP-144" (at 102.87 53.34 0)
+    (property "Footprint" "LQFP-144" (at 81.28 44.45 0)
       (effects (font (size 1.27 1.27) italic) hide)
     )
-    (property "Datasheet" "STM32H745ZIT6" (at 102.87 53.34 0)
+    (property "Datasheet" "STM32H745ZIT6" (at 81.28 44.45 0)
       (effects (font (size 1.27 1.27) italic) hide)
     )
@@
     )
   )
-  (symbol (lib_id "GAUL-Symboles:STM32-(STM32H745ZIT6)") (at 196.85 49.53 0) (unit 1)
+  (symbol (lib_id "Device:R") (at 44.45 93.98 180) (unit 1)
+    (in_bom yes) (on_board yes) (dnp no)
+    (property "Reference" "R10" (at 39.37 92.71 0)
+      (effects (font (size 1.27 1.27)) (justify right))
+    )
+    (property "Value" "170" (at 39.37 95.25 0)
+      (effects (font (size 1.27 1.27)) (justify right))
+    )
+    (property "Footprint" "" (at 46.228 93.98 90)
+      (effects (font (size 1.27 1.27)) hide)
+    )
+    (property "Datasheet" "~" (at 44.45 93.98 0)
+      (effects (font (size 1.27 1.27)) hide)
+    )
+    (pin "2")
+    (pin "1")
+    (instances
+      (project "Payload"
+        (path "/5f62c44b-34ee-4720-b187-b4a520863a8a"
+          (reference "R10") (unit 1)
+        )
+      )
+    )
+  )
+  (symbol (lib_id "Device:R") (at 50.8 96.52 180) (unit 1)
+    (in_bom yes) (on_board yes) (dnp no)
+    (property "Reference" "R12" (at 45.72 95.25 0)
+      (effects (font (size 1.27 1.27)) (justify right))
+    )
+    (property "Value" "170" (at 45.72 97.79 0)
+      (effects (font (size 1.27 1.27)) (justify right))
+    )
+    (property "Footprint" "" (at 52.578 96.52 90)
+      (effects (font (size 1.27 1.27)) hide)
+    )
+    (property "Datasheet" "~" (at 50.8 96.52 0)
+      (effects (font (size 1.27 1.27)) hide)
+    )
+    (pin "2")
+    (pin "1")
+    (instances
+      (project "Payload"
+        (path "/5f62c44b-34ee-4720-b187-b4a520863a8a"
+          (reference "R12") (unit 1)
+        )
+      )
+    )
+  )
+  (symbol (lib_id "GAUL-Symboles:STM32-(STM32H745ZIT6)") (at 189.23 34.29 0) (unit 1)
     (in_bom yes) (on_board yes) (dnp no) (fields_autoplaced)
-    (property "Reference" "U1" (at 227.33 39.37 0)
+    (property "Reference" "U1" (at 219.71 24.13 0)
       (effects (font (size 1.524 1.524)))
     )
-    (property "Value" "STM32-(STM32H745ZIT6)" (at 227.33 41.91 0)
+    (property "Value" "STM32-(STM32H745ZIT6)" (at 219.71 26.67 0)
       (effects (font (size 1.524 1.524)))
     )
-    (property "Footprint" "LQFP-144" (at 196.85 49.53 0)
+    (property "Footprint" "LQFP-144" (at 189.23 34.29 0)
       (effects (font (size 1.27 1.27) italic) hide)
     )
-    (property "Datasheet" "STM32H745ZIT6" (at 196.85 49.53 0)
+    (property "Datasheet" "STM32H745ZIT6" (at 189.23 34.29 0)
       (effects (font (size 1.27 1.27) italic) hide)
     )
@@
         )
       )
+    )
+  )
+  (symbol (lib_id "Device:R") (at 71.12 104.14 180) (unit 1)
+    (in_bom yes) (on_board yes) (dnp no)
+    (property "Reference" "R19" (at 66.04 102.87 0)
+      (effects (font (size 1.27 1.27)) (justify right))
+    )
+    (property "Value" "170" (at 66.04 105.41 0)
+      (effects (font (size 1.27 1.27)) (justify right))
+    )
+    (property "Footprint" "" (at 72.898 104.14 90)
+      (effects (font (size 1.27 1.27)) hide)
+    )
+    (property "Datasheet" "~" (at 71.12 104.14 0)
+      (effects (font (size 1.27 1.27)) hide)
+    )
+    (pin "2")
+    (pin "1")
+    (instances
+      (project "Payload"
+        (path "/5f62c44b-34ee-4720-b187-b4a520863a8a"
+          (reference "R19") (unit 1)
+        )
+      )
